File: avyortho.kicad_sch (KiCad schematic)
At the start: 99 parts, among them SW1 SW_Push_45deg, SW10 SW_Push_45deg, SW11 SW_Push_45deg, SW12 SW_Push_45deg, SW13 SW_Push_45deg, SW14 SW_Push_45deg, SW15 SW_Push_45deg, SW16 SW_Push_45deg, SW17 SW_Push_45deg, SW18 SW_Push_45deg, SW19 SW_Push_45deg, SW2 SW_Push_45deg, SW20 SW_Push_45deg, SW21 SW_Push_45deg, SW22 SW_Push_45deg, SW23 SW_Push_45deg, SW24 SW_Push_45deg, SW25 SW_Push_45deg, SW26 SW_Push_45deg, SW27 SW_Push_45deg, SW28 SW_Push_45deg, SW29 SW_Push_45deg, SW3 SW_Push_45deg, SW30 SW_Push_45deg, SW31 SW_Push_45deg, SW32 SW_Push_45deg, SW33 SW_Push_45deg, SW34 SW_Push_45deg, SW35 SW_Push_45deg, SW36 SW_Push_45deg, SW37 SW_Push_45deg, SW38 SW_Push_45deg, SW39 SW_Push_45deg, SW4 SW_Push_45deg, SW40 SW_Push_45deg, SW41 SW_Push_45deg, SW42 SW_Push_45deg, SW43 SW_Push_45deg, SW45 SW_Push_45deg, SW46 SW_Push_45deg, SW47 SW_Push_45deg, SW48 SW_Push_45deg, SW5 SW_Push_45deg, SW6 SW_Push_45deg, SW7 SW_Push_45deg, SW8 SW_Push_45deg, SW9 SW_Push_45deg, U3 XIAO-nRF52840-Plus-SMD

Commit message: layout pcb
Parts:
- D1, D10, D11, D12, D13, D14, D15, D16, D17, D18, D19, D2, D20, D21, D22, D23, D24, D25, D26, D27, D28, D29, D3, D30, D31, D32, D33, D34, D35, D36, D37, D38, D39, D4, D40, D41, D42, D43, D45, D46, D47, D48, D5, D6, D7, D8, D9: footprint (none) -> Diode_SMD:D_SOD-123
- R1, R2: footprint (none) -> Resistor_SMD:R_0805_2012Metric_Pad1.20x1.40mm_HandSolder
- SW1, SW10, SW11, SW12, SW13, SW14, SW15, SW16, SW17, SW18, SW19, SW2, SW20, SW21, SW22, SW23, SW24, SW25, SW26, SW27, SW28, SW29, SW3, SW30, SW31, SW32, SW33, SW34, SW35, SW36, SW37, SW38, SW39, SW4, SW40, SW41, SW42, SW43, SW45, SW46, SW47, SW48, SW5, SW6, SW7, SW8, SW9: footprint (none) -> PCM_marbastlib-mx:SW_MX_HS_KS-2P02B01-01_1u
- TP1, TP2: footprint (none) -> TestPoint:TestPoint_Pad_D3.0mm
- U3: footprint Seeed_Studio_XIAO_Series:XIAO-nRF52840-Plus-SMD -> Seeed Studio XIAO Series Library:XIAO-nRF52840-Plus-SMD
Connections:
- net COL6: no longer SW43.1
- net COL7: now also SW43.1
- no-connect marks 6 -> 7

Commit message: switch sockets to Kalih CPG151101S11-16 because available at lcsc
Parts:
- D1, D10, D11, D12, D13, D14, D15, D16, D17, D18, D19, D2, D20, D21, D22, D23, D24, D25, D26, D27, D28, D29, D3, D30, D31, D32, D33, D34, D35, D36, D37, D38, D39, D4, D40, D41, D42, D43, D45, D46, D47, D48, D5, D6, D7, D8, D9: MPN (none) -> 1N5819
- R1: MPN (none) -> CRCW0805806KFKEA
- R2: MPN (none) -> CRCW08052M00FKED
- SW1, SW10, SW11, SW12, SW13, SW14, SW15, SW16, SW17, SW18, SW19, SW2, SW20, SW21, SW22, SW23, SW24, SW25, SW26, SW27, SW28, SW29, SW3, SW30, SW31, SW32, SW33, SW34, SW35, SW36, SW37, SW38, SW39, SW4, SW40, SW41, SW42, SW43, SW45, SW46, SW47, SW48, SW5, SW6, SW7, SW8, SW9: footprint PCM_marbastlib-mx:SW_MX_HS_KS-2P02B01-01_1u -> PCM_marbastlib-mx:SW_MX_HS_CPG151101S11_1u; MPN (none) -> CPG151101S11-16
- U3: MPN (none) -> 102010672

Commit message: changes for submitting to half life prep week one
Parts:
- D1, D10, D11, D12, D13, D14, D15, D16, D17, D18, D19, D2, D20, D21, D22, D23, D24, D25, D26, D27, D28, D29, D3, D30, D31, D32, D33, D34, D35, D36, D37, D38, D39, D4, D40, D41, D42, D43, D45, D46, D47, D48, D5, D6, D7, D8, D9: MPN 1N5819 -> 1N4148W
- TP1, TP2: now left out of the parts list
